File: RP2040_AS3394.kicad_sch (KiCad schematic)
At the start: 41 parts, among them J1 Conn_01x03, J2 TYPE-C-31-M-12, J3 Conn_01x02, J4 Conn_01x08, J5 Conn_01x03, U1 RP2040, U2 NCP1117-3.3_SOT223, U3 W25Q128JVS, U7 TL071, Y1 X322512MSB4SI

Commit message: continuing work on second version
Connections:
- net AS3394_PWM/Out: now also C52.1, R16.1
- net GND: now also U7.3 (+)
Changed lines of the file:
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@@
   (junction (at 128.27 83.82) (diameter 0) (color 0 0 0 0)
+  )
+  (junction (at 162.56 142.24) (diameter 0) (color 0 0 0 0)
   )
   (junction (at 231.14 62.23) (diameter 0) (color 0 0 0 0)
@@
     (stroke (width 0) (type default) (color 0 0 0 0))
   )
-  (wire (pts (xy 162.56 119.38) (xy 162.56 137.16))
+  (wire (pts (xy 162.56 119.38) (xy 162.56 142.24))
     (stroke (width 0) (type default) (color 0 0 0 0))
   )
@@
     (stroke (width 0) (type default) (color 0 0 0 0))
   )
+  (wire (pts (xy 162.56 142.24) (xy 170.18 142.24))
+    (stroke (width 0) (type default) (color 0 0 0 0))
+  )
   (wire (pts (xy 243.84 72.39) (xy 247.65 72.39))
     (stroke (width 0) (type default) (color 0 0 0 0))
@@
     (stroke (width 0) (type default) (color 0 0 0 0))
   )
-  (wire (pts (xy 162.56 137.16) (xy 170.18 137.16))
-    (stroke (width 0) (type default) (color 0 0 0 0))
-  )
   (wire (pts (xy 62.23 88.9) (xy 62.23 78.74))
     (stroke (width 0) (type default) (color 0 0 0 0))
@@
     (stroke (width 0) (type default) (color 0 0 0 0))
   )
+  (wire (pts (xy 167.64 137.16) (xy 170.18 137.16))
+    (stroke (width 0) (type default) (color 0 0 0 0))
+  )
   (wire (pts (xy 246.38 107.95) (xy 246.38 109.22))
     (stroke (width 0) (type default) (color 0 0 0 0))
@@
     (stroke (width 0) (type default) (color 0 0 0 0))
   )
-  (wire (pts (xy 156.21 142.24) (xy 170.18 142.24))
+  (wire (pts (xy 156.21 142.24) (xy 162.56 142.24))
     (stroke (width 0) (type default) (color 0 0 0 0))
   )
@@
     )
     (property "Datasheet" "" (id 3) (at 182.88 153.67 0)
+      (effects (font (size 1.27 1.27)) hide)
+    )
+    (pin "1")
+  )
+  (symbol (lib_id "power:GND") (at 167.64 137.16 0) (unit 1)
+    (in_bom yes) (on_board yes)
+    (property "Reference" "#PWR0109" (id 0) (at 167.64 143.51 0)
+      (effects (font (size 1.27 1.27)) hide)
+    )
+    (property "Value" "GND" (id 1) (at 167.64 140.97 0))
+    (property "Footprint" "" (id 2) (at 167.64 137.16 0)
+      (effects (font (size 1.27 1.27)) hide)
+    )
+    (property "Datasheet" "" (id 3) (at 167.64 137.16 0)
       (effects (font (size 1.27 1.27)) hide)
     )
@@
       (reference "#PWR0108") (unit 1) (value "VEE") (footprint "")
     )
+    (path "/755a71c6-bd30-40cf-ab80-6f6e4fe965bd"
+      (reference "#PWR0109") (unit 1) (value "GND") (footprint "")
+    )
     (path "/0d7e14e3-8efa-45a6-8744-5aa07e3d3e44"
       (reference "C1") (unit 1) (value "100n") (footprint "Capacitor_SMD:C_0402_1005Metric")
@@
     )
     (path "/4be0f50f-df7d-4a82-b90c-e414038b561e/ddd76b89-2a88-4309-a333-bdf8de8cfe06"
-      (reference "D3") (unit 1) (value "D_Small") (footprint "Diode_SMD:D_SMA")
+      (reference "D3") (unit 1) (value "D_Small") (footprint "Diode_SMD:D_SOD-123")
     )
     (path "/4be0f50f-df7d-4a82-b90c-e414038b561e/27946d3c-8904-45e3-be89-3739e9e319a1"
-      (reference "D4") (unit 1) (value "D_Small") (footprint "Diode_SMD:D_SMA")
+      (reference "D4") (unit 1) (value "D_Small") (footprint "Diode_SMD:D_SOD-123")
     )
     (path "/4be0f50f-df7d-4a82-b90c-e414038b561e/d863356e-35a7-4549-89c4-1048508fa152"
-      (reference "D5") (unit 1) (value "D_Small") (footprint "Diode_SMD:D_SMA")
+      (reference "D5") (unit 1) (value "D_Small") (footprint "Diode_SMD:D_SOD-123")
     )
     (path "/4be0f50f-df7d-4a82-b90c-e414038b561e/e923455c-5904-4966-8e48-2190902b1404"
-      (reference "D6") (unit 1) (value "D_Small") (footprint "Diode_SMD:D_SMA")
+      (reference "D6") (unit 1) (value "D_Small") (footprint "Diode_SMD:D_SOD-123")
     )
     (path "/4be0f50f-df7d-4a82-b90c-e414038b561e/baa2fb89-4811-4d24-a01c-de8f2a48b73b"
