File: RP2040_AS3394.kicad_sch (KiCad schematic)
At the start: 38 parts, among them J1 Conn_01x03, J2 TYPE-C-31-M-12, J3 Conn_01x05, J4 Conn_01x09, U1 RP2040, U2 NCP1117-3.3_SOT223, U3 W25Q128JVS, U7 NCP1117-5.0_SOT223, Y1 X322512MSB4SI

Commit message: Updated to Kicad 7
Connections:
- no-connect marks 6 -> 19
